Commit message: updates

File: crab_model/description/crab_core.xacro (robot description, xacro)
@@ -4,16 +4,17 @@
     <xacro:include filename="colors.xacro"/>
     <xacro:include filename="inertial_macros.xacro"/>
-    <!-- BASE_FOOTPRINT LINK -->
-    <link name = "base_link"></link>
+    <xacro:include filename="crab_properties.xacro"/>
+    <!-- Wrold LINK -->
+    <link name = "world"></link>
+    <!-- BASE FOODPRINT AND JOINT -->
     <joint name = 'base_footprint_joint' type = "fixed">
         <origin xyz="0.0 0.0 0.0" rpy="0.0 0.0 0.0"/>
-        <parent link="base_link"/>
+        <parent link="world"/>
         <child link="base_footprint"/>
     </joint>
     <link name="base_footprint"></link>
-    <!-- BODY JOINT AND LINK -->
-    <!-- BODY joint will be made non fixed when the whole robot is ready-->
+    <!-- BODY LINK AND JOINT -->
     <joint name="body_joint" type="fixed">
-        <origin xyz="0.0 0.0 0.8" rpy="0.0 0.0 0.0"/>
+        <origin xyz="0.0 0.0 ${body_link_height}" rpy="0.0 0.0 0.0"/>
         <parent link="base_link"/>
         <child link="body_link"/>
@@ -23,8 +24,33 @@
             <origin xyz="0.0 0.0 0.0" rpy="0.0 0.2 0.0"/>
             <geometry>
-                <box size="0.5 0.3 0.05"/>
+                <box size="${body_link_x_dim} ${body_link_y_dim} ${body_link_z_dim}"/>
             </geometry>
             <material name="red"/>
         </visual>
     </link>
+    <!-- COXA LINK AND JOINTS -->
+    <joint name="coxa_joint_L" type="revolute">
+        <origin xyz="${coxa_joint_Ox} ${coxa_joint_Oy} ${coxa_joint_Oz}" rpy="0.0 -${pi/2} 0.0"/>
+        <parent link="body_link"/>
+        <child link="coxa_link_L"/>
+        <axis xyz="0 0 1"/>
+    </joint>
+    <link name="coxa_link_L">
+        <visual>
+            <origin xyz="${coxa_link_Ox} ${coxa_link_Oy} ${coxa_link_Oz}" rpy="0.0 ${coxa_link_Ry} 0.0"/>
+            <geometry>
+                <cylinder length="${coxa_link_length}" radius="${coxa_link_radius}"/>
+            </geometry>
+            <material name="blue"/>
+        </visual>
+        <xacro:inertial_cylinder mass="${coxa_link_mass}" length="${coxa_link_length}" radius="${coxa_link_radius}">
+            <origin xyz="${coxa_link_Ox} ${coxa_link_Oy} ${coxa_link_Oz}"/>
+        </xacro:inertial_cylinder>
+    </link>
+    <!-- BASIS LINK AND JOINTS -->
+    <!-- ISCHIUM LINK AND JOINT-->
+    <!-- MERUS LINK AND JOINT-->
+    <!-- CARPUS LINK AND JOINTS -->
+    <!-- MANUS LINK AND JOINT-->
+    <!-- DACTYL LINK AND JOINT-->
 </robot>

File: crab_model/description/crab_properties.xacro (robot description, xacro)
@@ -3,8 +3,8 @@
     <!-- Constant parameters -->
     <xacro:property name="body_link_mass" value="140.0" /> <!-- Kg -->
-    <xacro:property name="body_link_height" value="1.0" /> <!-- m -->
-    <xacro:property name="body_link_x_dim" value="0.55" /> <!-- m -->
-    <xacro:property name="body_link_y_dim" value="0.4" /> <!-- m -->
-    <xacro:property name="body_link_z_dim" value="0.3" /> <!-- m -->
+    <xacro:property name="body_link_height" value="0.8" /> <!-- m -->
+    <xacro:property name="body_link_x_dim" value="0.5" /> <!-- m -->
+    <xacro:property name="body_link_y_dim" value="0.3" /> <!-- m -->
+    <xacro:property name="body_link_z_dim" value="0.05" /> <!-- m -->
     <xacro:property name="coxa_link_mass" value="0.301" /> <!-- Kg -->
     <xacro:property name="coxa_joint_Ox" value="0.0" /> <!-- m -->
