Commit message: ros2control updates

File: crab_model/description/crab.xacro (robot description, xacro)
@@ -7,5 +7,6 @@
   <xacro:include filename="crab_properties.xacro"/>
   <xacro:include filename="crab_legs.xacro"/>
-  <xacro:include filename="gazebo_control.xacro"/>
+  <xacro:include filename="ros2_control_leg.xacro"/>
+  <xacro:include filename="ros2_control_crab.xacro"/>
   <!--BASE LINK-->
   <link name = "base_link"></link>
@@ -25,4 +26,6 @@
     </visual>
   </link>
+  <gazebo reference="body_link">
+    <material>Gazebo/Blue</material>
   <xacro:leg suffix="R1" reflect="1" Ox="0.3" Oy="0.3" Oz="0.0"/>
   <xacro:leg suffix="R2" reflect="1" Ox="0.3" Oy="0.0" Oz="0.0"/>
