Commit message: crab stl

File: crab_model/description/crab_properties.xacro (robot description, xacro)
@@ -2,5 +2,5 @@
 <robot xmlns:xacro="http://www.ros.org/wiki/xacro" >
     <!-- Constant parameters -->
-    <xacro:property name="body_link_mass" value="140.0" /> <!-- Kg -->
+    <xacro:property name="body_link_mass" value="1.0" /> <!-- Kg -->
     <xacro:property name="body_link_height" value="0.8" /> <!-- m -->
     <xacro:property name="body_link_x_dim" value="0.5" /> <!-- m -->
@@ -44,5 +44,5 @@
     <xacro:property name="manus_link_length" value="0.4" /> <!-- m -->
     <xacro:property name="manus_link_radius" value="0.05" /> <!-- m -->
-    <xacro:property name="dactyl_mass" value="0.001" /> <!-- Kg -->
+    <xacro:property name="dactyl_mass" value="0.01" /> <!-- Kg -->
     <xacro:property name="dactyl_radius" value="0.05" /> <!-- m -->
     <xacro:property name="dactyl_joint_Ox" value="0.0" /> <!-- m -->

File: crab_model/description/ros2_control_crab.xacro (robot description, xacro)
@@ -15,5 +15,4 @@
             </hardware>
         </xacro:unless>
-        <joint name = "" />
         <xacro:leg_control suffix="0"/>
         <xacro:leg_control suffix="1"/>
@@ -23,4 +22,5 @@
         <xacro:leg_control suffix="5"/>
     </ros2_control>
+    <!-- When not using Gazebo we need to run ros2 run controller_manager ros2_control_node -->
     <gazebo>
         <plugin name="gazebo_ros2_control" filename="libgazebo_ros2_control.so">
