Commit message: updates

File: crab_model/description/crab.urdf.xacro (robot description, xacro)
@@ -1,96 +1,9 @@
 <?xml version="1.0"?>
 <robot xmlns:xacro="http://www.ros.org/wiki/xacro" name="spider_crab">
-  <!-- 材质定义 -->
-  <material name="crab_red">
-    <color rgba="0.8 0.3 0.3 1"/>
-  </material>
-  <material name="crab_white">
-    <color rgba="0.9 0.9 0.9 1"/>
-  </material>
-  <!-- 常量 -->
-  <xacro:property name="body_radius" value="0.15"/>
-  <xacro:property name="body_length" value="0.2"/>
-  <xacro:property name="leg_length1" value="0.5"/>
-  <xacro:property name="leg_length2" value="0.4"/>
-  <xacro:property name="leg_length3" value="0.3"/>
-  <xacro:property name="leg_radius" value="0.02"/>
-  <xacro:property name="PI" value="3.1415926535897931"/>
-  <!-- 身体 -->
-  <link name="base_link">
-    <visual>
-      <geometry>
-        <sphere radius="${body_radius}"/>
-      </geometry>
-      <material name="crab_red"/>
-    </visual>
-  </link>
-  <!-- 腿宏定义：可按需要加更多关节 -->
-  <xacro:macro name="crab_leg" params="prefix angle">
-    <!-- 髋关节 -->
-    <joint name="${prefix}_hip_joint" type="revolute">
-      <parent link="base_link"/>
-      <child link="${prefix}_upper"/>
-      <origin xyz="${body_radius*cos(angle)} ${body_radius*sin(angle)} 0" rpy="0 0 ${angle}"/>
-      <axis xyz="0 0 1"/>
-      <limit lower="-1.5" upper="1.5" effort="10" velocity="2"/>
-    </joint>
-    <!-- 大腿 -->
-    <link name="${prefix}_upper">
-      <visual>
-        <geometry>
-          <cylinder radius="${leg_radius}" length="${leg_length1}"/>
-        </geometry>
-        <origin xyz="0 0 ${-leg_length1/2}" rpy="0 0 0"/>
-        <material name="crab_white"/>
-      </visual>
-    </link>
-    <!-- 膝关节 -->
-    <joint name="${prefix}_knee_joint" type="revolute">
-      <parent link="${prefix}_upper"/>
-      <child link="${prefix}_middle"/>
-      <origin xyz="0 0 ${-leg_length1}" rpy="0 0 0"/>
-      <axis xyz="0 1 0"/>
-      <limit lower="-2" upper="2" effort="10" velocity="2"/>
-    </joint>
-    <!-- 小腿 -->
-    <link name="${prefix}_middle">
-      <visual>
-        <geometry>
-          <cylinder radius="${leg_radius}" length="${leg_length2}"/>
-        </geometry>
-        <origin xyz="0 0 ${-leg_length2/2}" rpy="0 0 0"/>
-        <material name="crab_red"/>
-      </visual>
-    </link>
-    <!-- 脚关节&脚爪 -->
-    <joint name="${prefix}_ankle_joint" type="revolute">
-      <parent link="${prefix}_middle"/>
-      <child link="${prefix}_tip"/>
-      <origin xyz="0 0 ${-leg_length2}" rpy="0 0 0"/>
-      <axis xyz="0 1 0"/>
-      <limit lower="-2" upper="2" effort="10" velocity="2"/>
-    </joint>
-    <link name="${prefix}_tip">
-      <visual>
-        <geometry>
-          <cylinder radius="${leg_radius*0.8}" length="${leg_length3}"/>
-        </geometry>
-        <origin xyz="0 0 ${-leg_length3/2}" rpy="0 0 0"/>
-        <material name="crab_white"/>
-      </visual>
-    </link>
-  </xacro:macro>
-  <!-- 生成12条腿，分布在身体两侧，每30度一条 -->
-  <xacro:crab_leg prefix="leg1" angle="0"/>
-  <xacro:crab_leg prefix="leg2" angle="${PI/6}"/>
-  <xacro:crab_leg prefix="leg3" angle="${PI/3}"/>
-  <xacro:crab_leg prefix="leg4" angle="${PI/2}"/>
-  <xacro:crab_leg prefix="leg5" angle="${2*PI/3}"/>
-  <xacro:crab_leg prefix="leg6" angle="${5*PI/6}"/>
-  <xacro:crab_leg prefix="leg7" angle="${PI}"/>
-  <xacro:crab_leg prefix="leg8" angle="${7*PI/6}"/>
-  <xacro:crab_leg prefix="leg9" angle="${4*PI/3}"/>
-  <xacro:crab_leg prefix="leg10" angle="${3*PI/2}"/>
-  <xacro:crab_leg prefix="leg11" angle="${5*PI/3}"/>
-  <xacro:crab_leg prefix="leg12" angle="${11*PI/6}"/>
+  <xacro:arg name="use_ros2_control" default="false"/>
+  <xacro:arg name="sim_mode" default="true"/>
+  <xacro:include filename="crab_core.xacro"/>
+  <xacro:if value="$(arg use_ros2_control)">
+    <xacro:include filename="crab_ros2_control.xacro"/>
+  </xacro:if>
 </robot>

File: crab_model/description/crab_model_gazebo.xacro (robot description, xacro)
@@ -2,7 +2,7 @@
 <robot xmlns:xacro="http://ros.org/wiki/xacro" name="crab">
 <!-- Build the body frame -->
-	<link name="base_link" />
+	<link name="cam1" />
 	<joint name="base_joint" type="fixed">
-		<parent link="base_link" />
+		<parent link="cam1" />
 		<child link="thorax" />
 		<origin xyz="0 0 0" rpy="0 0 0" />

Commit message: rough crab model

File: crab_model/description/crab.urdf.xacro (robot description, xacro)
@@ -2,8 +2,31 @@
 <robot xmlns:xacro="http://www.ros.org/wiki/xacro" name="spider_crab">
   <xacro:arg name="use_ros2_control" default="false"/>
-  <xacro:arg name="sim_mode" default="true"/>
-  <xacro:include filename="crab_core.xacro"/>
-  <xacro:if value="$(arg use_ros2_control)">
-    <xacro:include filename="crab_ros2_control.xacro"/>
-  </xacro:if>
+  <xacro:arg name="use_sim_time" default="false"/>
+  <xacro:include filename="crab_legs.xacro"/>
+  <xacro:include filename="colors.xacro"/>
+  <xacro:include filename="inertial_macros.xacro"/>
+  <xacro:include filename="crab_properties.xacro"/>
+  <!--BASE LINK-->
+  <link name = "base_link"></link>
+  <!-- BODY JOINT AND LINK-->
+  <joint name="body_joint" type="fixed">
+    <parent link="base_link"/>
+    <child link="body_link"/>
+    <origin xyz="0 0 1.0" rpy="0 0 0"/>
+  </joint>
+  <link name ="body_link">
+    <visual>
+      <origin xyz="0 0 0" rpy="0 0 0"/>
+      <geometry>
+        <box size="0.5 1 0.15"/>
+      </geometry>
+      <material name="blue"/>
+    </visual>
+  </link>
+  <xacro:leg suffix="R1" reflect="1" Ox="0.3" Oy="0.3" Oz="0.0"/>
+  <xacro:leg suffix="R2" reflect="1" Ox="0.3" Oy="0.0" Oz="0.0"/>
+  <xacro:leg suffix="R3" reflect="1" Ox="0.3" Oy="-0.3" Oz="0.0"/>
+  <xacro:leg suffix="L1" reflect="-1" Ox="-0.3" Oy="0.3" Oz="0.0"/>
+  <xacro:leg suffix="L2" reflect="-1" Ox="-0.3" Oy="0.0" Oz="0.0"/>
+  <xacro:leg suffix="L3" reflect="-1" Ox="-0.3" Oy="-0.3" Oz="0.0"/>
 </robot>

File: crab_model/description/crab_legs.xacro (robot description, xacro)
@@ -2,4 +2,5 @@
 <robot xmlns:xacro="http://www.ros.org/wiki/xacro">
     <xacro:macro name="leg" params="suffix reflect Ox Oy Oz">
+        <!-- -->
         <!-- COXA JOINT AND LINK-->
         <joint name="coxa_joint_${suffix}" type="revolute">
@@ -7,5 +8,5 @@
                 <parent link="body_link"/>
                 <child link="coxa_link_${suffix}"/>
-                <limit effort="100" velocity="100.0" lower="-3.14" upper="3.14" />
+                <limit effort="250.0" velocity="10.0" lower="-3.14" upper="3.14" />
                 <axis xyz="0 0 1"/>
                 <dynamics damping="0.7"/>
@@ -13,5 +14,5 @@
         <link name="coxa_link_${suffix}">
             <visual>
-                <origin xyz="${coxa_link_Ox} ${reflect*coxa_link_Oy} ${coxa_link_Oz}" rpy="0.0 ${coxa_link_Ry} 0.0"/>
+                <origin xyz="${coxa_link_Ox} ${coxa_link_Oy} ${coxa_link_Oz}" rpy=" 0.0  ${coxa_link_Ry} 0.0"/>
                 <geometry>
                     <cylinder length="${coxa_link_length}" radius="${coxa_link_radius}"/>
@@ -19,67 +20,73 @@
                 <material name="red"/>
             </visual>
-            <collision>
-                <origin xyz="${coxa_link_Ox} ${coxa_link_Oy} ${coxa_link_Oz}" rpy="0.0 ${coxa_link_Ry} 0.0"/>
+        </link>
+        <!-- MERUS JOINT AND JOINT-->
+        <joint name="merus_joint_${suffix}" type="revolute">
+            <origin xyz="${reflect*merus_joint_Ox} ${merus_joint_Oy} ${merus_joint_Oz}" rpy="0.0 ${reflect*merus_joint_Ry} 0.0"/>
+            <parent link="coxa_link_${suffix}"/>
+            <child link="merus_link_${suffix}"/>
+            <limit effort="250.0" velocity="10.0" lower="-3.14" upper="3.14" />
+            <axis xyz="0 1 0"/>
+        </joint>
+        <link name="merus_link_${suffix}">
+            <visual>
+                <origin xyz="${merus_link_Ox} ${merus_link_Oy} ${merus_link_Oz}" rpy="0.0 0.0 0.0"/>
                 <geometry>
-                    <cylinder length="${coxa_link_length}" radius="${coxa_link_radius}"/>
+                    <cylinder length="${merus_link_length}" radius="${merus_link_radius}"/>
                 </geometry>
-            </collision>
-            <xacro:inertial_cylinder mass="${coxa_link_mass}" length="${coxa_link_length}" radius="${coxa_link_radius}">
-                <origin xyz="${coxa_link_Ox} ${coxa_link_Oy} ${coxa_link_Oz}" rpy="0.0 ${coxa_link_Ry} 0.0"/>
-            </xacro:inertial_cylinder>
+                <material name="blue"/>
+            </visual>
         </link>
-        <!-- FEMUR JOINT AND LINK-->
-        <joint name="femur_joint_${suffix}" type="revolute">
-            <origin xyz="${femur_joint_Ox} ${reflect*femur_joint_Oy} ${femur_joint_Oz}" rpy="0.0 ${femur_joint_Ry} 0.0"/>
-            <parent link="coxa_link_${suffix}"/>
-            <child link="femur_link_${suffix}"/>
-            <limit effort="100" velocity="100.0" lower="-3.14" upper="3.14" />
-            <axis xyz="0 0 ${reflect}"/>
+        <!-- CARPUS JOINT AND LINK-->
+        <joint name="carpus_joint_${suffix}" type="revolute">
+            <origin xyz="${carpus_joint_Ox} ${carpus_joint_Oy} ${carpus_joint_Oz}" rpy="0.0 ${reflect*carpus_joint_Ry} 0.0"/>
+            <parent link="merus_link_${suffix}"/>
+            <child link="carpus_link_${suffix}"/>
+            <limit effort="250.0" velocity="10.0" lower="-3.14" upper="3.14" />
+            <axis xyz="${reflect} 0 0"/>
             <dynamics damping="0.7"/>
         </joint>
-        <link name="femur_link_${suffix}">
+        <link name="carpus_link_${suffix}">
             <visual>
-                <origin xyz="${femur_link_Ox} 0.0 0.0" rpy="0.0 0.0 0.0"/>
+                <origin xyz="${carpus_link_Ox} ${carpus_link_Oy} ${carpus_link_Oz}" rpy="0.0 0.0 0.0"/>
                 <geometry>
-                    <box size="${femur_link_dx} ${femur_link_dy} ${femur_link_dz}"/>
+                    <cylinder length="${carpus_link_length}" radius = "${carpus_link_radius}"/>
                 </geometry>
-                <material name="orange"/>
+                <material name="red"/>
             </visual>
-            <collision>
-                <origin xyz="${femur_link_Ox} 0.0 0.0" rpy="0.0 0.0 0.0"/>
-                <geometry>
-                    <box size="${femur_link_dx} ${femur_link_dy} ${femur_link_dz}"/>
-                </geometry>
-            </collision>
-            <xacro:inertial_box mass="${femur_link_mass}" x="${femur_link_dx}" y="${femur_link_dy}" z='${femur_link_dz}'>
-                <origin xyz="${femur_link_Ox} 0.0 0.0" rpy="0.0 0.0 0.0"/>
-            </xacro:inertial_box>
         </link>
-        <!-- TIBIA JOINT AND LINK -->
-        <joint name="tibia_joint_${suffix}" type="revolute">
-            <origin xyz="${tibia_joint_Ox} ${tibia_joint_Oy} ${tibia_joint_Oz}" rpy="0.0 0.0 0.0"/>
-            <parent link="femur_link_${suffix}"/>
-            <child link="tibia_link_${suffix}"/>
-            <limit effort="100" velocity="100.0" lower="-3.14" upper="3.14" />
-            <axis xyz="0 0 ${reflect}"/>
+        <!-- MANUS JOINT AND LINK -->
+        <joint name="manus_joint_${suffix}" type="revolute">
+            <origin xyz="${manus_joint_Ox} ${manus_joint_Oy} ${manus_joint_Oz}" rpy="0.0 ${reflect*manus_joint_Ry} 0.0"/>
+            <parent link="carpus_link_${suffix}"/>
+            <child link="manus_link_${suffix}"/>
+            <limit effort="250.0" velocity="10.0" lower="-3.14" upper="3.14" />
+            <axis xyz="0 1 0"/>
             <dynamics damping="0.7"/>
         </joint>
-        <link name="tibia_link_${suffix}">
+        <link name="manus_link_${suffix}">
             <visual>
-                <origin xyz="${tibia_link_Ox} 0.0 0.0" rpy="0.0 0.0 0.0"/>
+                <origin xyz="0.0 0.0 ${manus_link_Oz}" rpy="0.0 0.0 0.0"/>
                 <geometry>
-                    <box size="${tibia_link_dx} ${tibia_link_dy} ${tibia_link_dz}"/>
+                    <cylinder length="${manus_link_length}" radius = "${manus_link_radius}"/>
                 </geometry>
-                <material name="black"/>
+                <material name="blue"/>
             </visual>
-            <collision>
-                <origin xyz="${tibia_link_Ox} 0.0 0.0" rpy="0.0 0.0 0.0"/>
+        </link>
+        <!-- DACTYL JOINT AND LINK-->
+        <joint name="dactyl_joint_${suffix}" type="fixed">
+            <origin xyz="0.0 0.0 -${manus_link_length}" rpy="0.0 0.0 0.0"/>
+            <parent link="manus_link_${suffix}"/>
+            <child link="dactyl_link_${suffix}"/>
+            <dynamics damping="0.7"/>
+        </joint>
+        <link name="dactyl_link_${suffix}">
+            <visual>
+                <origin xyz="${dactyl_link_Ox} ${dactyl_link_Oy} ${dactyl_link_Oz}" rpy="0.0 0.0 0.0"/>
                 <geometry>
-                    <box size="${tibia_link_dx} ${tibia_link_dy} ${tibia_link_dz}"/>
+                    <sphere radius="${dactyl_radius}"/>
                 </geometry>
-            </collision>
-            <xacro:inertial_box mass="${tibia_link_mass}" x="${tibia_link_dx}" y="${tibia_link_dy}" z="${tibia_link_dz}">
-                <origin xyz="${tibia_link_Ox} 0.0 0.0" rpy="0.0 0.0 0.0"/>
-            </xacro:inertial_box>
+                <material name="red"/>
+            </visual>
         </link>
     </xacro:macro>

File: crab_model/description/crab_properties.xacro (robot description, xacro)
@@ -8,43 +8,48 @@
     <xacro:property name="body_link_z_dim" value="0.05" /> <!-- m -->
     <xacro:property name="coxa_link_mass" value="0.301" /> <!-- Kg -->
-    <xacro:property name="coxa_joint_Ox" value="0.0" /> <!-- m -->
-    <xacro:property name="coxa_joint_Oy" value="0.0" /> <!-- m -->
-    <xacro:property name="coxa_joint_Oz" value="0.0" /> <!-- m -->
-    <xacro:property name="coxa_link_Ox" value="0.03" /> <!-- m -->
-    <xacro:property name="coxa_link_Oy" value="-0.05" /> <!-- m -->
-    <xacro:property name="coxa_link_Oz" value="-0.05" /> <!-- m -->
-    <xacro:property name="coxa_link_Ry" value="1.57" /> <!-- rad -->
+    <xacro:property name="coxa_link_Ox" value="0.0" /> <!-- m -->
+    <xacro:property name="coxa_link_Oy" value="0.0" /> <!-- m -->
+    <xacro:property name="coxa_link_Oz" value="0.0" /> <!-- m -->
+    <xacro:property name="coxa_link_Ry" value="-1.57" /> <!-- rad -->
     <xacro:property name="coxa_link_length" value="0.1" /> <!-- m -->
     <xacro:property name="coxa_link_radius" value="0.05" /> <!-- m -->
-    <xacro:property name="femur_link_mass" value="0.501" /> <!-- Kg -->
-    <xacro:property name="femur_joint_Ox" value="0.07" /> <!-- m -->
-    <xacro:property name="femur_joint_Oy" value="-0.05" /> <!-- m -->
-    <xacro:property name="femur_joint_Oz" value="-0.05" /> <!-- m -->
-    <xacro:property name="femur_joint_Ry" value="-1.57" /> <!-- rad -->
-    <xacro:property name="femur_link_Ox" value="0.0" /> <!-- m -->
-    <xacro:property name="femur_link_Oy" value="-0.15" /> <!-- m -->
-    <xacro:property name="femur_link_Oz" value="-0.03" /> <!-- m -->
-    <xacro:property name="femur_link_dx" value="0.03" /> <!-- m -->
-    <xacro:property name="femur_link_dy" value="0.3" /> <!-- m -->
-    <xacro:property name="femur_link_dz" value="0.01" /> <!-- m -->
-    <xacro:property name="tibia_link_mass" value="0.401" /> <!-- Kg -->
-    <xacro:property name="tibia_joint_Ox" value="0.0" /> <!-- m -->
-    <xacro:property name="tibia_joint_Oy" value="-0.3" /> <!-- m -->
-    <xacro:property name="tibia_joint_Oz" value="-0.01" /> <!-- m -->
-    <xacro:property name="tibia_link_Ry" value="3.14" /> <!-- rad -->
-    <xacro:property name="tibia_link_Ox" value="0.0" /> <!-- m -->
-    <xacro:property name="tibia_link_Oy" value="-0.15" /> <!-- m -->
-    <xacro:property name="tibia_link_Oz" value="0.0" /> <!-- m -->
-    <xacro:property name="tibia_link_dx" value="0.03" /> <!-- m -->
-    <xacro:property name="tibia_link_dy" value="-0.27" /> <!-- m -->
-    <xacro:property name="tibia_link_dz" value="0.01" /> <!-- m -->
-    <xacro:property name="foot_mass" value="0.001" /> <!-- Kg -->
-    <xacro:property name="foot_radius" value="0.025" /> <!-- m -->
-    <xacro:property name="foot_joint_Ox" value="0.0" /> <!-- m -->
-    <xacro:property name="foot_joint_Oy" value="-0.295" /> <!-- m -->
-    <xacro:property name="foot_joint_Oz" value="0.0" /> <!-- m -->
-    <xacro:property name="foot_joint_Rz" value="0.0" /> <!-- rad -->
-    <xacro:property name="foot_link_Ox" value="0.0" /> <!-- m -->
-    <xacro:property name="foot_link_Oy" value="0.0" /> <!-- m -->
-    <xacro:property name="foot_link_Oz" value="0.0" /> <!-- m -->
+    <xacro:property name="merus_link_mass" value="0.501" /> <!-- Kg -->
+    <xacro:property name="merus_joint_Ox" value="0.05" /> <!-- m -->
+    <xacro:property name="merus_joint_Oy" value="0.0" /> <!-- m -->
+    <xacro:property name="merus_joint_Oz" value="0.0" /> <!-- m -->
+    <xacro:property name="merus_joint_Ry" value="-1.92" /> <!-- rad -->
+    <xacro:property name="merus_link_Ox" value="0.0" /> <!-- m -->
+    <xacro:property name="merus_link_Oy" value="0.0" /> <!-- m -->
+    <xacro:property name="merus_link_Oz" value="-0.2" /> <!-- m -->
+    <xacro:property name="merus_link_length" value="0.4" /> <!-- m -->
+    <xacro:property name="merus_link_radius" value="0.05" /> <!-- m -->
+    <xacro:property name="carpus_link_mass" value="0.501" /> <!-- Kg -->
+    <xacro:property name="carpus_joint_Ox" value="0.0" /> <!-- m -->
+    <xacro:property name="carpus_joint_Oy" value="0.0" /> <!-- m -->
+    <xacro:property name="carpus_joint_Oz" value="-0.45" /> <!-- m -->
+    <xacro:property name="carpus_joint_Ry" value="1.0" /> <!-- rad -->
+    <xacro:property name="carpus_link_Ox" value="0.0" /> <!-- m -->
+    <xacro:property name="carpus_link_Oy" value="0.0" /> <!-- m -->
+    <xacro:property name="carpus_link_Oz" value="-0.1" /> <!-- m -->
+    <xacro:property name="carpus_link_length" value="0.2" /> <!-- m -->
+    <xacro:property name="carpus_link_radius" value="0.05" /> <!-- m -->
+    <xacro:property name="manus_link_mass" value="0.501" /> <!-- Kg -->
+    <xacro:property name="manus_joint_Ox" value="0.0" /> <!-- m -->
+    <xacro:property name="manus_joint_Oy" value="0.0" /> <!-- m -->
+    <xacro:property name="manus_joint_Oz" value="-0.2" /> <!-- m -->
+    <xacro:property name="manus_joint_Ry" value="0.17" /> <!-- rad -->
+    <xacro:property name="manus_link_Ox" value="0.0" /> <!-- m -->
+    <xacro:property name="manus_link_Oy" value="0.0" /> <!-- m -->
+    <xacro:property name="manus_link_Oz" value="-0.2" /> <!-- m -->
+    <xacro:property name="manus_link_length" value="0.4" /> <!-- m -->
+    <xacro:property name="manus_link_radius" value="0.05" /> <!-- m -->
+    <xacro:property name="dactyl_mass" value="0.001" /> <!-- Kg -->
+    <xacro:property name="dactyl_radius" value="0.05" /> <!-- m -->
+    <xacro:property name="dactyl_joint_Ox" value="0.0" /> <!-- m -->
+    <xacro:property name="dactyl_joint_Oy" value="0.0" /> <!-- m -->
+    <xacro:property name="dactyl_joint_Oz" value="0.0" /> <!-- m -->
+    <xacro:property name="dactyl_joint_Rz" value="0.0" /> <!-- rad -->
+    <xacro:property name="dactyl_link_Ox" value="0.0" /> <!-- m -->
+    <xacro:property name="dactyl_link_Oy" value="0.0" /> <!-- m -->
+    <xacro:property name="dactyl_link_Oz" value="-0.025" /> <!-- m -->
 </robot>

Commit message: ros2_control updates

File: crab_model/description/crab.urdf.xacro (robot description, xacro)
@@ -3,8 +3,9 @@
   <xacro:arg name="use_ros2_control" default="false"/>
   <xacro:arg name="use_sim_time" default="false"/>
-  <xacro:include filename="crab_legs.xacro"/>
   <xacro:include filename="colors.xacro"/>
   <xacro:include filename="inertial_macros.xacro"/>
   <xacro:include filename="crab_properties.xacro"/>
+  <xacro:include filename="crab_legs.xacro"/>
+  <xacro:include filename="gazebo_control.xacro"/>
   <!--BASE LINK-->
   <link name = "base_link"></link>

File: crab_model/description/crab_legs.xacro (robot description, xacro)
@@ -21,4 +21,7 @@
             </visual>
         </link>
+        <gazebo reference = "coxa_link_${suffix}">
+            <material>Gazebo/Red</material>
+        </gazebo>
         <!-- MERUS JOINT AND JOINT-->
         <joint name="merus_joint_${suffix}" type="revolute">
@@ -38,4 +41,7 @@
             </visual>
         </link>
+        <gazebo reference = "coxa_link_${suffix}">
+            <material>Gazebo/Blue</material>
+        </gazebo>
         <!-- CARPUS JOINT AND LINK-->
         <joint name="carpus_joint_${suffix}" type="revolute">
@@ -56,4 +62,7 @@
             </visual>
         </link>
+        <gazebo reference = "coxa_link_${suffix}">
+            <material>Gazebo/Red</material>
+        </gazebo>
         <!-- MANUS JOINT AND LINK -->
         <joint name="manus_joint_${suffix}" type="revolute">
@@ -74,4 +83,7 @@
             </visual>
         </link>
+        <gazebo reference = "coxa_link_${suffix}">
+            <material>Gazebo/Blue</material>
+        </gazebo>
         <!-- DACTYL JOINT AND LINK-->
         <joint name="dactyl_joint_${suffix}" type="fixed">
@@ -90,4 +102,7 @@
             </visual>
         </link>
+        <gazebo reference = "coxa_link_${suffix}">
+            <material>Gazebo/Red</material>
+        </gazebo>
     </xacro:macro>
 </robot>
