Commit message: gazebo

File: crab_model/description/crab.urdf.xacro (robot description, xacro)
@@ -2,11 +2,9 @@
 <robot xmlns:xacro="http://www.ros.org/wiki/xacro" name="spider_crab">
   <xacro:arg name="use_ros2_control" default="false"/>
-  <xacro:arg name="use_sim_time" default="false"/>
+  <xacro:arg name="use_sim_time" default="true"/>
   <xacro:include filename="colors.xacro"/>
   <xacro:include filename="inertial_macros.xacro"/>
   <xacro:include filename="crab_properties.xacro"/>
   <xacro:include filename="crab_legs.xacro"/>
-  <xacro:include filename="ros2_control_leg.xacro"/>
-  <xacro:include filename="ros2_control_crab.xacro"/>
   <!--BASE LINK-->
   <link name = "base_link"></link>
@@ -15,5 +13,5 @@
     <parent link="base_link"/>
     <child link="body_link"/>
-    <origin xyz="0 0 1.0" rpy="0 0 0"/>
+    <origin xyz="0 0 0.26" rpy="0 0 0"/>
   </joint>
   <link name ="body_link">
@@ -25,7 +23,17 @@
       <material name="blue"/>
     </visual>
+    <collision>
+      <origin xyz="0 0 0" rpy="0 0 0"/>
+      <geometry>
+        <box size="0.5 1 0.15"/>
+      </geometry>
+    </collision>
+    <xacro:inertial_box mass="1.0" x="0.5" y="1.0" z="0.15">
+      <origin xyz="0 0 0" rpy="0 0 0"/>
+    </xacro:inertial_box>
   </link>
   <gazebo reference="body_link">
     <material>Gazebo/Blue</material>
+  </gazebo>
   <xacro:leg suffix="R1" reflect="1" Ox="0.3" Oy="0.3" Oz="0.0"/>
   <xacro:leg suffix="R2" reflect="1" Ox="0.3" Oy="0.0" Oz="0.0"/>

File: crab_model/description/crab_legs.xacro (robot description, xacro)
@@ -20,4 +20,13 @@
                 <material name="red"/>
             </visual>
+            <collision>
+                <origin xyz="${coxa_link_Ox} ${coxa_link_Oy} ${coxa_link_Oz}" rpy=" 0.0  ${coxa_link_Ry} 0.0"/>
+                <geometry>
+                    <cylinder length="${coxa_link_length}" radius="${coxa_link_radius}"/>
+                </geometry>
+            </collision>
+            <xacro:inertial_cylinder mass="${coxa_link_mass}" length="${coxa_link_length}" radius="${coxa_link_radius}">
+                <origin xyz="${coxa_link_Ox} ${coxa_link_Oy} ${coxa_link_Oz}" rpy=" 0.0  ${coxa_link_Ry} 0.0"/>
+            </xacro:inertial_cylinder>
         </link>
         <gazebo reference = "coxa_link_${suffix}">
@@ -40,4 +49,13 @@
                 <material name="blue"/>
             </visual>
+            <collision>
+                <origin xyz="${merus_link_Ox} ${merus_link_Oy} ${merus_link_Oz}" rpy="0.0 0.0 0.0"/>
+                <geometry>
+                    <cylinder length="${merus_link_length}" radius="${merus_link_radius}"/>
+                </geometry>
+            </collision>
+            <xacro:inertial_cylinder mass="${merus_link_mass}" length="${merus_link_length}" radius="${merus_link_radius}">
+                <origin xyz="${merus_link_Ox} ${merus_link_Oy} ${merus_link_Oz}" rpy="0.0 0.0 0.0"/>
+            </xacro:inertial_cylinder>
         </link>
         <gazebo reference = "coxa_link_${suffix}">
@@ -61,4 +79,13 @@
                 <material name="red"/>
             </visual>
+            <collision>
+                <origin xyz="${carpus_link_Ox} ${carpus_link_Oy} ${carpus_link_Oz}" rpy="0.0 0.0 0.0"/>
+                <geometry>
+                    <cylinder length="${carpus_link_length}" radius = "${carpus_link_radius}"/>
+                </geometry>
+            </collision>
+            <xacro:inertial_cylinder mass="${carpus_link_mass}" length="${carpus_link_length}" radius="${carpus_link_radius}">
+                <origin xyz="${carpus_link_Ox} ${carpus_link_Oy} ${carpus_link_Oz}" rpy="0.0 0.0 0.0"/>
+            </xacro:inertial_cylinder>
         </link>
         <gazebo reference = "coxa_link_${suffix}">
@@ -82,4 +109,13 @@
                 <material name="blue"/>
             </visual>
+            <collision>
+                <origin xyz="0.0 0.0 ${manus_link_Oz}" rpy="0.0 0.0 0.0"/>
+                <geometry>
+                    <cylinder length="${manus_link_length}" radius = "${manus_link_radius}"/>
+                </geometry>
+            </collision>
+            <xacro:inertial_cylinder mass="${manus_link_mass}" length="${manus_link_length}" radius="${manus_link_radius}">
+                <origin xyz="0.0 0.0 ${manus_link_Oz}" rpy="0.0 0.0 0.0"/>
+            </xacro:inertial_cylinder>
         </link>
         <gazebo reference = "coxa_link_${suffix}">
@@ -101,4 +137,13 @@
                 <material name="red"/>
             </visual>
+            <collision>
+                <origin xyz="${dactyl_link_Ox} ${dactyl_link_Oy} ${dactyl_link_Oz}" rpy="0.0 0.0 0.0"/>
+                <geometry>
+                    <sphere radius="${dactyl_radius}"/>
+                </geometry>
+            </collision>
+            <xacro:inertial_sphere mass="${dactyl_mass}" radius="${dactyl_radius}">
+                <origin xyz="${dactyl_link_Ox} ${dactyl_link_Oy} ${dactyl_link_Oz}" rpy="0.0 0.0 0.0"/>
+            </xacro:inertial_sphere>
         </link>
         <gazebo reference = "coxa_link_${suffix}">

Commit message: ros2control

File: crab_model/description/crab.urdf.xacro (robot description, xacro)
@@ -7,4 +7,7 @@
   <xacro:include filename="crab_properties.xacro"/>
   <xacro:include filename="crab_legs.xacro"/>
+  <xacro:include filename="gazebo_control.xacro"/>
+  <xacro:include filename="ros2_control_crab.xacro"/>
+  <xacro:include filename="ros2_control_leg.xacro"/>
   <!--BASE LINK-->
   <link name = "base_link"></link>
@@ -95,12 +98,3 @@
   <xacro:leg suffix="R3" reflect="-1" Ox="-0.14" Oy="-0.09" Oz="0.0" merus_link_length="0.16" carpus_link_length="0.07" manus_link_length ="0.10" fore_leg_Rz="0.0" dactyl="1" scale_x="0.001" scale_y="0.001" scale_z="0.006"/>
   <xacro:leg suffix="R4" reflect="-1" Ox="-0.18" Oy="-0.075" Oz="0.0" merus_link_length="0.13" carpus_link_length="0.058" manus_link_length ="0.09" fore_leg_Rz="0.0" dactyl="1" scale_x="0.001" scale_y="0.001" scale_z="0.005"/>
-  <gazebo reference="body_link">
-    <material>Gazebo/Red</material>
-  </gazebo>
-  <gazebo reference="eyes_left">
-    <material>Gazebo/Black</material>
-  </gazebo>
-  <gazebo reference="eyes_right">
-    <material>Gazebo/Black</material>
-  </gazebo>
 </robot>

File: crab_model/description/crab_legs.xacro (robot description, xacro)
@@ -159,7 +159,10 @@
         <!-- Gazebo material for all links -->
         <gazebo reference = "coxa_link_${suffix}">
-            <material>Gazebo/blue</material>
+            <material>Gazebo/Blue</material>
         </gazebo>
         <gazebo reference = "merus_link_${suffix}">
+            <material>Gazebo/Blue</material>
+        </gazebo>
+        <gazebo reference = "carpus_link_${suffix}">
             <material>Gazebo/Blue</material>
         </gazebo>

File: crab_model/description/ros2_control_crab.xacro (robot description, xacro)
@@ -7,4 +7,5 @@
             </hardware>
         </xacro:if>
+        <!-- If not using Gazebo, use Dynamixel hardware plugin -->
         <xacro:unless value="${arg use_sim_time}">
             <hardware>
@@ -15,10 +16,14 @@
             </hardware>
         </xacro:unless>
-        <xacro:leg_control suffix="0"/>
-        <xacro:leg_control suffix="1"/>
-        <xacro:leg_control suffix="2"/>
-        <xacro:leg_control suffix="3"/>
-        <xacro:leg_control suffix="4"/>
-        <xacro:leg_control suffix="5"/>
+        <xacro:leg_control suffix="F1"/>
+        <xacro:leg_control suffix="F2"/>
+        <xacro:leg_control suffix="L1"/>
+        <xacro:leg_control suffix="L2"/>
+        <xacro:leg_control suffix="L3"/>
+        <xacro:leg_control suffix="L4"/>
+        <xacro:leg_control suffix="R1"/>
+        <xacro:leg_control suffix="R2"/>
+        <xacro:leg_control suffix="R3"/>
+        <xacro:leg_control suffix="R4"/>
     </ros2_control>
     <!-- When not using Gazebo we need to run ros2 run controller_manager ros2_control_node -->

Commit message: new

File: crab_model/description/crab.urdf.xacro (robot description, xacro)
@@ -7,7 +7,6 @@
   <xacro:include filename="crab_properties.xacro"/>
   <xacro:include filename="crab_legs.xacro"/>
-  <xacro:include filename="gazebo_control.xacro"/>
+  <xacro:include filename="ros2_control_leg.xacro"/>
   <xacro:include filename="ros2_control_crab.xacro"/>
-  <xacro:include filename="ros2_control_leg.xacro"/>
   <!--BASE LINK-->
   <link name = "base_link"></link>
@@ -25,5 +24,6 @@
         <!-- Connect the two origins of ELlipsoids-->
         <!-- The center of body locates at the intersection of the large Ellipsoid and the staight line-->
-        <mesh filename="package://crab_model/meshes/crab_body.stl" scale="0.01 0.01 0.01"/>
+        <box size="0.27 0.20 0.1"/>
+        <!-- mesh filename="package://crab_model/meshes/crab_body.stl" scale="0.01 0.01 0.01"/ -->
       </geometry>
       <material name="red"/>
@@ -32,5 +32,6 @@
       <origin xyz="0 0 0" rpy="0 0 0"/>
       <geometry>
-        <mesh filename="package://crab_model/meshes/crab_body.stl" scale="0.01 0.01 0.01"/>
+        <box size="0.27 0.20 0.1"/>
+        <!-- mesh filename="package://crab_model/meshes/crab_body.stl" scale="0.01 0.01 0.01"/ -->
       </geometry>
     </collision>
@@ -86,4 +87,13 @@
     </xacro:inertial_box>
   </link>
+  <gazebo reference="body_link">
+      <material>Gazebo/Red</material>
+  </gazebo>
+  <gazebo reference="eyes_left">
+      <material>Gazebo/Black</material>
+  </gazebo>
+  <gazebo reference="eyes_right">
+      <material>Gazebo/Black</material>
+  </gazebo>
   <!-- CRAB LEGS-->
   <!-- reflect=1 means left side-->

File: crab_model/description/crab_legs.xacro (robot description, xacro)
@@ -157,4 +157,19 @@
             </link>
         </xacro:unless>
+        <gazebo reference = "coxa_link_${suffix}">
+            <material>Gazebo/Blue</material>
+        </gazebo>
+        <gazebo reference = "merus_link_${suffix}">
+            <material>Gazebo/Blue</material>
+        </gazebo>
+        <gazebo reference = "carpus_link_${suffix}">
+            <material>Gazebo/Blue</material>
+        </gazebo>
+        <gazebo reference = "manus_link_${suffix}">
+            <material>Gazebo/Blue</material>
+        </gazebo>
+        <gazebo reference = "dactyl_link_${suffix}">
+            <material>Gazebo/Blue</material>
+        </gazebo>
     </xacro:macro>
 </robot>

File: crab_model/description/ros2_control_crab.xacro (robot description, xacro)
@@ -1,4 +1,5 @@
 <?xml version="1.0"?>
 <robot xmlns:xacro="http://www.ros.org/wiki/xacro" >
+    <xacro:include filename="ros2_control_leg.xacro"/>
     <ros2_control name="GazeboSystem" type = "system">
         <xacro:if value="${arg use_sim_time}">
@@ -28,3 +29,9 @@
         <xacro:leg_control suffix="R4"/>
     </ros2_control>
+    <!-- ros_control plugin -->
+    <gazebo>
+      <plugin filename="libgazebo_ros2_control.so" name="gazebo_ros2_control">
+        <parameters>$(find crab_model)/config/my_controller.yaml</parameters>
+      </plugin>
+    </gazebo>
 </robot>

File: crab_model/description/ros2_control_leg.xacro (robot description, xacro)
@@ -3,5 +3,5 @@
     <xacro:macro name="leg_control" params="suffix">
         <joint name="coxa_joint_${suffix}">
-            <param name="id">${suffix*3 + 0}</param>
+            <param name="id">${suffix}</param>
             <param name="pos_kp">5000</param>
             <param name="pos_ki">1</param>
@@ -45,5 +45,5 @@
             <state_interface name="effort"/>
         </joint>
-        <joint name="femur_joint_${suffix}">
+        <joint name="merus_joint_${suffix}">
             <param name="id">${suffix*3 + 1}</param>
             <param name="pos_kp">5000</param>
@@ -70,5 +70,55 @@
             <state_interface name="effort"/>
         </joint>
-        <joint name="tibia_joint_${suffix}">
+        <joint name="carpus_joint_${suffix}">
+            <param name="id">${suffix}</param>
+            <param name="pos_kp">5000</param>
+            <param name="pos_ki">1</param>
+            <param name="pos_kd">3</param>
+            <param name="pos_max_integral_error">10000</param>
+            <command_interface name="position_pid">
+            <!--command_interface name="position"-->
+                <param name="min">-3.14</param>
+                <param name="max">3.14</param>
+            </command_interface>
+            <command_interface name="velocity">
+                <!--param name="min">-1.0</param>
+                <param name="max">1.0</param-->
+            </command_interface>
+            <xacro:if value="$(arg sim_mode)">
+                <command_interface name="effort"/>
+            </xacro:if>
+            <!--state_interface name="position"/-->
+            <state_interface name="position">
+                <param name="initial_value">2.3</param>
+            </state_interface>
+            <state_interface name="velocity"/>
+            <state_interface name="effort"/>
+        </joint>
+        <joint name="manus_joint_${suffix}">
+            <param name="id">${suffix*3 + 2}</param>
+            <param name="pos_kp">5000</param>
+            <param name="pos_ki">1</param>
+            <param name="pos_kd">3</param>
+            <param name="pos_max_integral_error">10000</param>
+            <command_interface name="position_pid">
+            <!--command_interface name="position"-->
+                <param name="min">-3.14</param>
+                <param name="max">3.14</param>
+            </command_interface>
+            <command_interface name="velocity">
+                <!--param name="min">-1.0</param>
+                <param name="max">1.0</param-->
+            </command_interface>
+            <xacro:if value="$(arg sim_mode)">
+                <command_interface name="effort"/>
+            </xacro:if>
+            <!--state_interface name="position"/-->
+            <state_interface name="position">
+                <param name="initial_value">2.3</param>
+            </state_interface>
+            <state_interface name="velocity"/>
+            <state_interface name="effort"/>
+        </joint>
+        <joint name="dactyl_joint_${suffix}">
             <param name="id">${suffix*3 + 2}</param>
             <param name="pos_kp">5000</param>
