Commit message: crab urdf model update

File: crab_model/description/crab_legs.xacro (robot description, xacro)
@@ -1,6 +1,6 @@
 <?xml version="1.0"?>
 <robot xmlns:xacro="http://www.ros.org/wiki/xacro">
-    <xacro:macro name="leg" params="suffix reflect Ox Oy Oz">
-        <!-- -->
+    <!-- FORE LEGS -->
+    <xacro:macro name="leg" params="suffix reflect Ox Oy Oz merus_link_length carpus_link_length manus_link_length fore_leg_Rz dactyl scale_x scale_y scale_z">
         <!-- COXA JOINT AND LINK-->
         <joint name="coxa_joint_${suffix}" type="revolute">
@@ -18,5 +18,5 @@
                     <cylinder length="${coxa_link_length}" radius="${coxa_link_radius}"/>
                 </geometry>
-                <material name="red"/>
+                <material name="blue"/>
             </visual>
             <collision>
@@ -30,18 +30,15 @@
             </xacro:inertial_cylinder>
         </link>
-        <gazebo reference = "coxa_link_${suffix}">
-            <material>Gazebo/Red</material>
-        </gazebo>
         <!-- MERUS JOINT AND JOINT-->
         <joint name="merus_joint_${suffix}" type="revolute">
-            <origin xyz="${reflect*merus_joint_Ox} ${merus_joint_Oy} ${merus_joint_Oz}" rpy="0.0 ${reflect*merus_joint_Ry} 0.0"/>
+            <origin xyz="${merus_joint_Ox} ${reflect*merus_joint_Oy} ${merus_joint_Oz}" rpy="${reflect*merus_joint_Rx} 0.0 0.0"/>
             <parent link="coxa_link_${suffix}"/>
             <child link="merus_link_${suffix}"/>
             <limit effort="250.0" velocity="10.0" lower="-3.14" upper="3.14" />
-            <axis xyz="0 1 0"/>
+            <axis xyz="1 0 0"/>
         </joint>
         <link name="merus_link_${suffix}">
             <visual>
-                <origin xyz="${merus_link_Ox} ${merus_link_Oy} ${merus_link_Oz}" rpy="0.0 0.0 0.0"/>
+                <origin xyz="${merus_link_Ox} ${merus_link_Oy} ${merus_link_length/2}" rpy="0.0 0.0 0.0"/>
                 <geometry>
                     <cylinder length="${merus_link_length}" radius="${merus_link_radius}"/>
@@ -50,5 +47,5 @@
             </visual>
             <collision>
-                <origin xyz="${merus_link_Ox} ${merus_link_Oy} ${merus_link_Oz}" rpy="0.0 0.0 0.0"/>
+                <origin xyz="${merus_link_Ox} ${merus_link_Oy} ${merus_link_length/2}" rpy="0.0 0.0 0.0"/>
                 <geometry>
                     <cylinder length="${merus_link_length}" radius="${merus_link_radius}"/>
@@ -56,13 +53,10 @@
             </collision>
             <xacro:inertial_cylinder mass="${merus_link_mass}" length="${merus_link_length}" radius="${merus_link_radius}">
-                <origin xyz="${merus_link_Ox} ${merus_link_Oy} ${merus_link_Oz}" rpy="0.0 0.0 0.0"/>
+                <origin xyz="${merus_link_Ox} ${merus_link_Oy} ${merus_link_length/2}" rpy="0.0 0.0 0.0"/>
             </xacro:inertial_cylinder>
         </link>
-        <gazebo reference = "coxa_link_${suffix}">
-            <material>Gazebo/Blue</material>
-        </gazebo>
         <!-- CARPUS JOINT AND LINK-->
         <joint name="carpus_joint_${suffix}" type="revolute">
-            <origin xyz="${carpus_joint_Ox} ${carpus_joint_Oy} ${carpus_joint_Oz}" rpy="0.0 ${reflect*carpus_joint_Ry} 0.0"/>
+            <origin xyz="${carpus_joint_Ox} ${carpus_joint_Oy} ${merus_link_length+carpus_link_radius}" rpy="${reflect*carpus_joint_Rx} 0.0 ${reflect*fore_leg_Rz}"/>
             <parent link="merus_link_${suffix}"/>
             <child link="carpus_link_${suffix}"/>
@@ -73,5 +67,5 @@
         <link name="carpus_link_${suffix}">
             <visual>
-                <origin xyz="${carpus_link_Ox} ${carpus_link_Oy} ${carpus_link_Oz}" rpy="0.0 0.0 0.0"/>
+                <origin xyz="${carpus_link_Ox} ${carpus_link_Oy} ${carpus_link_length/2}" rpy="0.0 0.0 0.0"/>
                 <geometry>
                     <cylinder length="${carpus_link_length}" radius = "${carpus_link_radius}"/>
@@ -80,5 +74,5 @@
             </visual>
             <collision>
-                <origin xyz="${carpus_link_Ox} ${carpus_link_Oy} ${carpus_link_Oz}" rpy="0.0 0.0 0.0"/>
+                <origin xyz="${carpus_link_Ox} ${carpus_link_Oy} ${carpus_link_length/2}" rpy="0.0 0.0 0.0"/>
                 <geometry>
                     <cylinder length="${carpus_link_length}" radius = "${carpus_link_radius}"/>
@@ -86,13 +80,10 @@
             </collision>
             <xacro:inertial_cylinder mass="${carpus_link_mass}" length="${carpus_link_length}" radius="${carpus_link_radius}">
-                <origin xyz="${carpus_link_Ox} ${carpus_link_Oy} ${carpus_link_Oz}" rpy="0.0 0.0 0.0"/>
+                <origin xyz="${carpus_link_Ox} ${carpus_link_Oy} ${carpus_link_length/2}" rpy="0.0 0.0 0.0"/>
             </xacro:inertial_cylinder>
         </link>
-        <gazebo reference = "coxa_link_${suffix}">
-            <material>Gazebo/Red</material>
-        </gazebo>
         <!-- MANUS JOINT AND LINK -->
         <joint name="manus_joint_${suffix}" type="revolute">
-            <origin xyz="${manus_joint_Ox} ${manus_joint_Oy} ${manus_joint_Oz}" rpy="0.0 ${reflect*manus_joint_Ry} 0.0"/>
+            <origin xyz="${manus_joint_Ox} ${manus_joint_Oy} ${carpus_link_length}" rpy="${reflect*manus_joint_Rx} 0.0 0.0"/>
             <parent link="carpus_link_${suffix}"/>
             <child link="manus_link_${suffix}"/>
@@ -103,5 +94,5 @@
         <link name="manus_link_${suffix}">
             <visual>
-                <origin xyz="0.0 0.0 ${manus_link_Oz}" rpy="0.0 0.0 0.0"/>
+                <origin xyz="0.0 0.0 ${manus_link_length/2}" rpy="0.0 0.0 0.0"/>
                 <geometry>
                     <cylinder length="${manus_link_length}" radius = "${manus_link_radius}"/>
@@ -110,5 +101,5 @@
             </visual>
             <collision>
-                <origin xyz="0.0 0.0 ${manus_link_Oz}" rpy="0.0 0.0 0.0"/>
+                <origin xyz="0.0 0.0 ${manus_link_length/2}" rpy="0.0 0.0 0.0"/>
                 <geometry>
                     <cylinder length="${manus_link_length}" radius = "${manus_link_radius}"/>
@@ -116,37 +107,66 @@
             </collision>
             <xacro:inertial_cylinder mass="${manus_link_mass}" length="${manus_link_length}" radius="${manus_link_radius}">
-                <origin xyz="0.0 0.0 ${manus_link_Oz}" rpy="0.0 0.0 0.0"/>
+                <origin xyz="0.0 0.0 ${manus_link_length/2}" rpy="0.0 0.0 0.0"/>
             </xacro:inertial_cylinder>
         </link>
-        <gazebo reference = "coxa_link_${suffix}">
-            <material>Gazebo/Blue</material>
-        </gazebo>
         <!-- DACTYL JOINT AND LINK-->
         <joint name="dactyl_joint_${suffix}" type="fixed">
-            <origin xyz="0.0 0.0 -${manus_link_length}" rpy="0.0 0.0 0.0"/>
+            <origin xyz="0.0 0.0 ${manus_link_length}" rpy="0.0 0.0 0.0"/>
             <parent link="manus_link_${suffix}"/>
             <child link="dactyl_link_${suffix}"/>
             <dynamics damping="0.7"/>
         </joint>
-        <link name="dactyl_link_${suffix}">
-            <visual>
-                <origin xyz="${dactyl_link_Ox} ${dactyl_link_Oy} ${dactyl_link_Oz}" rpy="0.0 0.0 0.0"/>
-                <geometry>
-                    <sphere radius="${dactyl_radius}"/>
-                </geometry>
-                <material name="red"/>
-            </visual>
-            <collision>
-                <origin xyz="${dactyl_link_Ox} ${dactyl_link_Oy} ${dactyl_link_Oz}" rpy="0.0 0.0 0.0"/>
-                <geometry>
-                    <sphere radius="${dactyl_radius}"/>
-                </geometry>
-            </collision>
-            <xacro:inertial_sphere mass="${dactyl_mass}" radius="${dactyl_radius}">
-                <origin xyz="${dactyl_link_Ox} ${dactyl_link_Oy} ${dactyl_link_Oz}" rpy="0.0 0.0 0.0"/>
-            </xacro:inertial_sphere>
-        </link>
+        <xacro:if value="${dactyl == 1}">
+            <link name="dactyl_link_${suffix}">
+                <visual>
+                    <origin xyz="${dactyl_link_Ox} ${dactyl_link_Oy} ${dactyl_link_Oz}" rpy="0.0 0.0 0.0"/>
+                    <geometry>
+                        <mesh filename="package://crab_model/meshes/dactyl.stl" scale="${scale_x} ${scale_y} ${scale_z}"/>
+                    </geometry>
+                    <material name="red"/>
+                </visual>
+                <collision>
+                    <origin xyz="${dactyl_link_Ox} ${dactyl_link_Oy} ${dactyl_link_Oz}" rpy="0.0 0.0 0.0"/>
+                    <geometry>
+                        <mesh filename="package://crab_model/meshes/dactyl.stl" scale="${scale_x} ${scale_y} ${scale_z}"/>
+                    </geometry>
+                </collision>
+                <xacro:inertial_sphere mass="${dactyl_mass}" radius="${dactyl_radius}">
+                    <origin xyz="${dactyl_link_Ox} ${dactyl_link_Oy} ${dactyl_link_Oz}" rpy="0.0 0.0 0.0"/>
+                </xacro:inertial_sphere>
+            </link>
+        </xacro:if>
+        <xacro:unless value="${dactyl == 1}">
+            <link name="dactyl_link_${suffix}">
+                <visual>
+                    <origin xyz="${dactyl_link_Ox} ${dactyl_link_Oy} ${dactyl_link_Oz}" rpy="0.0 0.0 0.0"/>
+                    <geometry>
+                        <mesh filename="package://crab_model/meshes/crab_claw.stl" scale="${scale_x} ${scale_y} ${scale_z}"/>
+                    </geometry>
+                    <material name="red"/>
+                </visual>
+                <collision>
+                    <origin xyz="${dactyl_link_Ox} ${dactyl_link_Oy} ${dactyl_link_Oz}" rpy="0.0 0.0 0.0"/>
+                    <geometry>
+                        <mesh filename="package://crab_model/meshes/crab_claw.stl" scale="${scale_x} ${scale_y} ${scale_z}"/>
+                    </geometry>
+                </collision>
+                <xacro:inertial_sphere mass="${dactyl_mass}" radius="${dactyl_radius}">
+                    <origin xyz="${dactyl_link_Ox} ${dactyl_link_Oy} ${dactyl_link_Oz}" rpy="0.0 0.0 0.0"/>
+                </xacro:inertial_sphere>
+            </link>
+        </xacro:unless>
+        <!-- Gazebo material for all links -->
         <gazebo reference = "coxa_link_${suffix}">
-            <material>Gazebo/Red</material>
+            <material>Gazebo/blue</material>
+        </gazebo>
+        <gazebo reference = "merus_link_${suffix}">
+            <material>Gazebo/Blue</material>
+        </gazebo>
+        <gazebo reference = "manus_link_${suffix}">
+            <material>Gazebo/Blue</material>
+        </gazebo>
+        <gazebo reference = "dactyl_link_${suffix}">
+            <material>Gazebo/Blue</material>
         </gazebo>
     </xacro:macro>

File: crab_model/description/crab_properties.xacro (robot description, xacro)
@@ -3,8 +3,8 @@
     <!-- Constant parameters -->
     <xacro:property name="body_link_mass" value="1.0" /> <!-- Kg -->
-    <xacro:property name="body_link_height" value="0.8" /> <!-- m -->
-    <xacro:property name="body_link_x_dim" value="0.5" /> <!-- m -->
-    <xacro:property name="body_link_y_dim" value="0.3" /> <!-- m -->
-    <xacro:property name="body_link_z_dim" value="0.05" /> <!-- m -->
+    <xacro:property name="body_link_height" value="0.3" /> <!-- m -->
+    <xacro:property name="body_link_Rx" value="0.0" /> <!-- rad -->
+    <xacro:property name="body_link_Ry" value="0.0" /> <!-- rad -->
+    <xacro:property name="body_link_Rz" value="0.0" /> <!-- rad -->
     <xacro:property name="coxa_link_mass" value="0.301" /> <!-- Kg -->
     <xacro:property name="coxa_link_Ox" value="0.0" /> <!-- m -->
@@ -12,44 +12,41 @@
     <xacro:property name="coxa_link_Oz" value="0.0" /> <!-- m -->
     <xacro:property name="coxa_link_Ry" value="-1.57" /> <!-- rad -->
-    <xacro:property name="coxa_link_length" value="0.1" /> <!-- m -->
-    <xacro:property name="coxa_link_radius" value="0.05" /> <!-- m -->
+    <xacro:property name="coxa_link_length" value="0.015" /> <!-- m -->
+    <xacro:property name="coxa_link_radius" value="0.015" /> <!-- m -->
     <xacro:property name="merus_link_mass" value="0.501" /> <!-- Kg -->
-    <xacro:property name="merus_joint_Ox" value="0.05" /> <!-- m -->
-    <xacro:property name="merus_joint_Oy" value="0.0" /> <!-- m -->
+    <xacro:property name="merus_joint_Ox" value="0.0" /> <!-- m -->
+    <xacro:property name="merus_joint_Oy" value="${coxa_link_radius}" /> <!-- m -->
     <xacro:property name="merus_joint_Oz" value="0.0" /> <!-- m -->
-    <xacro:property name="merus_joint_Ry" value="-1.92" /> <!-- rad -->
+    <xacro:property name="merus_joint_Rx" value="-1.1" /> <!-- rad -->
     <xacro:property name="merus_link_Ox" value="0.0" /> <!-- m -->
     <xacro:property name="merus_link_Oy" value="0.0" /> <!-- m -->
-    <xacro:property name="merus_link_Oz" value="-0.2" /> <!-- m -->
-    <xacro:property name="merus_link_length" value="0.4" /> <!-- m -->
-    <xacro:property name="merus_link_radius" value="0.05" /> <!-- m -->
+    <xacro:property name="merus_link_Oz" value="0.0"/> <!-- m -->
+    <xacro:property name="merus_link_radius" value="0.015" /> <!-- m -->
     <xacro:property name="carpus_link_mass" value="0.501" /> <!-- Kg -->
     <xacro:property name="carpus_joint_Ox" value="0.0" /> <!-- m -->
     <xacro:property name="carpus_joint_Oy" value="0.0" /> <!-- m -->
-    <xacro:property name="carpus_joint_Oz" value="-0.45" /> <!-- m -->
-    <xacro:property name="carpus_joint_Ry" value="1.0" /> <!-- rad -->
+    <xacro:property name="carpus_joint_Oz" value="0.0" /> <!-- m -->
+    <xacro:property name="carpus_joint_Rx" value="-1.57" /> <!-- rad -->
     <xacro:property name="carpus_link_Ox" value="0.0" /> <!-- m -->
     <xacro:property name="carpus_link_Oy" value="0.0" /> <!-- m -->
-    <xacro:property name="carpus_link_Oz" value="-0.1" /> <!-- m -->
-    <xacro:property name="carpus_link_length" value="0.2" /> <!-- m -->
-    <xacro:property name="carpus_link_radius" value="0.05" /> <!-- m -->
+    <xacro:property name="carpus_link_Oz" value="0.0" /> <!-- m -->
+    <xacro:property name="carpus_link_radius" value="0.015" /> <!-- m -->
     <xacro:property name="manus_link_mass" value="0.501" /> <!-- Kg -->
     <xacro:property name="manus_joint_Ox" value="0.0" /> <!-- m -->
     <xacro:property name="manus_joint_Oy" value="0.0" /> <!-- m -->
-    <xacro:property name="manus_joint_Oz" value="-0.2" /> <!-- m -->
-    <xacro:property name="manus_joint_Ry" value="0.17" /> <!-- rad -->
+    <xacro:property name="manus_joint_Oz" value="0.0" /> <!-- m -->
+    <xacro:property name="manus_joint_Rx" value="-0.087" /> <!-- rad -->
     <xacro:property name="manus_link_Ox" value="0.0" /> <!-- m -->
     <xacro:property name="manus_link_Oy" value="0.0" /> <!-- m -->
-    <xacro:property name="manus_link_Oz" value="-0.2" /> <!-- m -->
-    <xacro:property name="manus_link_length" value="0.4" /> <!-- m -->
-    <xacro:property name="manus_link_radius" value="0.05" /> <!-- m -->
+    <xacro:property name="manus_link_Oz" value="0.0" /> <!-- m -->
+    <xacro:property name="manus_link_radius" value="0.015" /> <!-- m -->
     <xacro:property name="dactyl_mass" value="0.01" /> <!-- Kg -->
-    <xacro:property name="dactyl_radius" value="0.05" /> <!-- m -->
+    <xacro:property name="dactyl_radius" value="0.015" /> <!-- m -->
     <xacro:property name="dactyl_joint_Ox" value="0.0" /> <!-- m -->
     <xacro:property name="dactyl_joint_Oy" value="0.0" /> <!-- m -->
     <xacro:property name="dactyl_joint_Oz" value="0.0" /> <!-- m -->
-    <xacro:property name="dactyl_joint_Rz" value="0.0" /> <!-- rad -->
+    <xacro:property name="dactyl_joint_Ry" value="0.0" /> <!-- rad -->
     <xacro:property name="dactyl_link_Ox" value="0.0" /> <!-- m -->
     <xacro:property name="dactyl_link_Oy" value="0.0" /> <!-- m -->
-    <xacro:property name="dactyl_link_Oz" value="-0.025" /> <!-- m -->
+    <xacro:property name="dactyl_link_Oz" value="0.0" /> <!-- m -->
 </robot>

Commit message: ros2control

File: crab_model/description/crab_legs.xacro (robot description, xacro)
@@ -157,20 +157,4 @@
             </link>
         </xacro:unless>
-        <!-- Gazebo material for all links -->
-        <gazebo reference = "coxa_link_${suffix}">
-            <material>Gazebo/Blue</material>
-        </gazebo>
-        <gazebo reference = "merus_link_${suffix}">
-            <material>Gazebo/Blue</material>
-        </gazebo>
-        <gazebo reference = "carpus_link_${suffix}">
-            <material>Gazebo/Blue</material>
-        </gazebo>
-        <gazebo reference = "manus_link_${suffix}">
-            <material>Gazebo/Blue</material>
-        </gazebo>
-        <gazebo reference = "dactyl_link_${suffix}">
-            <material>Gazebo/Blue</material>
-        </gazebo>
     </xacro:macro>
 </robot>

File: crab_model/description/gazebo_control.xacro (robot description, xacro)
@@ -28,5 +28,5 @@
     <gazebo>
       <plugin filename="libgazebo_ros2_control.so" name="gazebo_ros2_control">
-        <parameters>$(find crab_model)/config/gaz_ros2_control.yaml</parameters>
+        <parameters>$(find crab_model)/config/my_controller.yaml</parameters>
       </plugin>
     </gazebo>

File: crab_model/description/ros2_control_crab.xacro (robot description, xacro)
@@ -4,4 +4,5 @@
         <xacro:if value="${arg use_sim_time}">
             <hardware>
+                <!--Receive msg from controller-->
                 <plugin>gazebo_ros2_control/GazeboSystem</plugin>
             </hardware>
@@ -27,9 +28,3 @@
         <xacro:leg_control suffix="R4"/>
     </ros2_control>
-    <!-- When not using Gazebo we need to run ros2 run controller_manager ros2_control_node -->
-    <gazebo>
-        <plugin name="gazebo_ros2_control" filename="libgazebo_ros2_control.so">
-            <parameters>$(find crab_model/config/gazebo_control.yaml)</parameters>
-        </plugin>
-    </gazebo>
 </robot>
