Commit message: update readme

File: crab_model/description/crab_legs.xacro (robot description, xacro)
@@ -14,5 +14,5 @@
         <link name="coxa_link_${suffix}">
             <visual>
-                <origin xyz="${coxa_link_Ox} ${coxa_link_Oy} ${coxa_link_Oz}" rpy=" 0.0  ${coxa_link_Ry} 0.0"/>
+                <origin xyz="${coxa_link_Ox} ${coxa_link_Oy} ${coxa_link_Oz}" rpy=" 0.0  0.0 0.0"/>
                 <geometry>
                     <cylinder length="${coxa_link_length}" radius="${coxa_link_radius}"/>
@@ -21,5 +21,5 @@
             </visual>
             <collision>
-                <origin xyz="${coxa_link_Ox} ${coxa_link_Oy} ${coxa_link_Oz}" rpy=" 0.0  ${coxa_link_Ry} 0.0"/>
+                <origin xyz="${coxa_link_Ox} ${coxa_link_Oy} ${coxa_link_Oz}" rpy=" 0.0  0.0 0.0"/>
                 <geometry>
                     <cylinder length="${coxa_link_length}" radius="${coxa_link_radius}"/>
@@ -122,5 +122,5 @@
                     <origin xyz="${dactyl_link_Ox} ${dactyl_link_Oy} ${dactyl_link_Oz}" rpy="0.0 0.0 0.0"/>
                     <geometry>
-                        <mesh filename="package://crab_model/meshes/dactyl.stl" scale="${scale_x} ${scale_y} ${scale_z}"/>
+                        <mesh filename="file://$(find crab_model)/meshes/dactyl.stl" scale="${scale_x} ${scale_y} ${scale_z}"/>
                     </geometry>
                     <material name="red"/>
@@ -129,5 +129,5 @@
                     <origin xyz="${dactyl_link_Ox} ${dactyl_link_Oy} ${dactyl_link_Oz}" rpy="0.0 0.0 0.0"/>
                     <geometry>
-                        <mesh filename="package://crab_model/meshes/dactyl.stl" scale="${scale_x} ${scale_y} ${scale_z}"/>
+                        <mesh filename="file://$(find crab_model)/meshes/dactyl.stl" scale="${scale_x} ${scale_y} ${scale_z}"/>
                     </geometry>
                 </collision>
@@ -142,5 +142,5 @@
                     <origin xyz="${dactyl_link_Ox} ${dactyl_link_Oy} ${dactyl_link_Oz}" rpy="0.0 0.0 0.0"/>
                     <geometry>
-                        <mesh filename="package://crab_model/meshes/crab_claw.stl" scale="${scale_x} ${scale_y} ${scale_z}"/>
+                        <mesh filename="file://$(find crab_model)/meshes/crab_claw.stl" scale="${scale_x} ${scale_y} ${scale_z}"/>
                     </geometry>
                     <material name="red"/>
@@ -149,5 +149,5 @@
                     <origin xyz="${dactyl_link_Ox} ${dactyl_link_Oy} ${dactyl_link_Oz}" rpy="0.0 0.0 0.0"/>
                     <geometry>
-                        <mesh filename="package://crab_model/meshes/crab_claw.stl" scale="${scale_x} ${scale_y} ${scale_z}"/>
+                        <mesh filename="file://$(find crab_model)/meshes/crab_claw.stl" scale="${scale_x} ${scale_y} ${scale_z}"/>
                     </geometry>
                 </collision>

File: crab_model/description/crab_properties.xacro (robot description, xacro)
@@ -3,5 +3,5 @@
     <!-- Constant parameters -->
     <xacro:property name="body_link_mass" value="1.0" /> <!-- Kg -->
-    <xacro:property name="body_link_height" value="0.3" /> <!-- m -->
+    <xacro:property name="body_link_height" value="0.15" /> <!-- m -->
     <xacro:property name="body_link_Rx" value="0.0" /> <!-- rad -->
     <xacro:property name="body_link_Ry" value="0.0" /> <!-- rad -->

File: crab_model/description/ros2_control_leg.xacro (robot description, xacro)
@@ -1,5 +1,6 @@
 <?xml version="1.0"?>
 <robot xmlns:xacro="http://www.ros.org/wiki/xacro">
-    <xacro:macro name="leg_control" params="suffix">
+    <!--relfect ==1 == left-->
+    <xacro:macro name="leg_control" params="suffix reflect">
         <joint name="coxa_joint_${suffix}">
             <param name="id">${suffix}</param>
@@ -8,37 +9,13 @@
             <param name="pos_kd">3</param>
             <param name="pos_max_integral_error">10000</param>
-            <command_interface name="position_pid">
-            <!--command_interface name="position"-->
-                <param name="min">-3.14</param>
-                <param name="max">3.14</param>
-            </command_interface>
-            <command_interface name="velocity">
-                <!--param name="min">-1.0</param>
-                <param name="max">1.0</param-->
-            </command_interface>
-            <xacro:if value="$(arg sim_mode)">
-                <command_interface name="effort"/>
-            </xacro:if>
-            <!--state_interface name="position"/-->
+            <param name="min">-3.14</param>
+            <param name="max">3.14</param>
+            <command_interface name="position"/>
+            <command_interface name="position_pid"/>
+            <command_interface name="velocity"/>
+            <command_interface name="effort"/>
             <!--SET INITIAL POSITION, note that this will not reset when gazebo world is restarted-->
             <state_interface name="position">
-                <xacro:if value="${suffix==0}">
-                    <param name="initial_value">0.75</param>
-                </xacro:if>
-                <xacro:if value="${suffix==1}">
-                    <param name="initial_value">0.0</param>
-                </xacro:if>
-                <xacro:if value="${suffix==2}">
-                    <param name="initial_value">-0.75</param>
-                </xacro:if>
-                <xacro:if value="${suffix==3}">
-                    <param name="initial_value">-0.75</param>
-                </xacro:if>
-                <xacro:if value="${suffix==4}">
-                    <param name="initial_value">0.0</param>
-                </xacro:if>
-                <xacro:if value="${suffix==5}">
-                    <param name="initial_value">0.75</param>
-                </xacro:if>
+                <param name="initial_value">0.0</param>
             </state_interface>
             <state_interface name="velocity"/>
@@ -46,24 +23,17 @@
         </joint>
         <joint name="merus_joint_${suffix}">
-            <param name="id">${suffix*3 + 1}</param>
+            <param name="id">${suffix}</param>
             <param name="pos_kp">5000</param>
             <param name="pos_ki">1</param>
             <param name="pos_kd">3</param>
             <param name="pos_max_integral_error">10000</param>
-            <command_interface name="position_pid">
-            <!--command_interface name="position"-->
-                <param name="min">-3.14</param>
-                <param name="max">3.14</param>
-            </command_interface>
-            <command_interface name="velocity">
-                <!--param name="min">-1.0</param>
-                <param name="max">1.0</param-->
-            </command_interface>
-            <xacro:if value="$(arg sim_mode)">
-                <command_interface name="effort"/>
-            </xacro:if>
-            <!--state_interface name="position"/-->
+            <param name="min">-3.14</param>
+            <param name="max">3.14</param>
+            <command_interface name="position"/>
+            <command_interface name="position_pid"/>
+            <command_interface name="velocity"/>
+            <command_interface name="effort"/>
             <state_interface name="position">
-                <param name="initial_value">0.8</param>
+                <param name="initial_value">0.0</param>
             </state_interface>
             <state_interface name="velocity"/>
@@ -76,19 +46,12 @@
             <param name="pos_kd">3</param>
             <param name="pos_max_integral_error">10000</param>
-            <command_interface name="position_pid">
-            <!--command_interface name="position"-->
-                <param name="min">-3.14</param>
-                <param name="max">3.14</param>
-            </command_interface>
-            <command_interface name="velocity">
-                <!--param name="min">-1.0</param>
-                <param name="max">1.0</param-->
-            </command_interface>
-            <xacro:if value="$(arg sim_mode)">
-                <command_interface name="effort"/>
-            </xacro:if>
-            <!--state_interface name="position"/-->
+            <param name="min">-3.14</param>
+            <param name="max">3.14</param>
+            <command_interface name="position"/>
+            <command_interface name="position_pid"/>
+            <command_interface name="velocity"/>
+            <command_interface name="effort"/>
             <state_interface name="position">
-                <param name="initial_value">2.3</param>
+                <param name="initial_value">0.0</param>
             </state_interface>
             <state_interface name="velocity"/>
@@ -96,49 +59,17 @@
         </joint>
         <joint name="manus_joint_${suffix}">
-            <param name="id">${suffix*3 + 2}</param>
+            <param name="id">${suffix}</param>
             <param name="pos_kp">5000</param>
             <param name="pos_ki">1</param>
             <param name="pos_kd">3</param>
             <param name="pos_max_integral_error">10000</param>
-            <command_interface name="position_pid">
-            <!--command_interface name="position"-->
-                <param name="min">-3.14</param>
-                <param name="max">3.14</param>
-            </command_interface>
-            <command_interface name="velocity">
-                <!--param name="min">-1.0</param>
-                <param name="max">1.0</param-->
-            </command_interface>
-            <xacro:if value="$(arg sim_mode)">
-                <command_interface name="effort"/>
-            </xacro:if>
-            <!--state_interface name="position"/-->
+            <param name="min">-3.14</param>
+            <param name="max">3.14</param>
+            <command_interface name="position"/>
+            <command_interface name="position_pid"/>
+            <command_interface name="velocity"/>
+            <command_interface name="effort"/>
             <state_interface name="position">
-                <param name="initial_value">2.3</param>
-            </state_interface>
-            <state_interface name="velocity"/>
-            <state_interface name="effort"/>
-        </joint>
-        <joint name="dactyl_joint_${suffix}">
-            <param name="id">${suffix*3 + 2}</param>
-            <param name="pos_kp">5000</param>
-            <param name="pos_ki">1</param>
-            <param name="pos_kd">3</param>
-            <param name="pos_max_integral_error">10000</param>
-            <command_interface name="position_pid">
-            <!--command_interface name="position"-->
-                <param name="min">-3.14</param>
-                <param name="max">3.14</param>
-            </command_interface>
-            <command_interface name="velocity">
-                <!--param name="min">-1.0</param>
-                <param name="max">1.0</param-->
-            </command_interface>
-            <xacro:if value="$(arg sim_mode)">
-                <command_interface name="effort"/>
-            </xacro:if>
-            <!--state_interface name="position"/-->
-            <state_interface name="position">
-                <param name="initial_value">2.3</param>
+                <param name="initial_value">0.0</param>
             </state_interface>
             <state_interface name="velocity"/>
